Commit message: Starting to split files according to Gazebo tutorial.

File: defs/pioneer3dx_wheel.xacro (robot description, xacro)
@@ -59,9 +59,9 @@
   </collision>
   </link>
-  <transmission type="pr2_mechanism_model/SimpleTransmission" name="${parent}_${suffix}_wheel_trans">
+<!--   <transmission type="pr2_mechanism_model/SimpleTransmission" name="${parent}_${suffix}_wheel_trans">
     <actuator name="base_${suffix}_wheel_motor" />
     <joint name="base_${suffix}_wheel_joint" />
     <mechanicalReduction>${reflect * 624/35 * 80/19}</mechanicalReduction>
-  </transmission>
+  </transmission> -->
   <joint name="base_${suffix}_wheel_joint" type="continuous">
     <axis xyz="0 1 0"/>

File: urdf/pioneer3dx.xacro (robot description, xacro)
@@ -2,9 +2,5 @@
 <!-- Orignal in ucs-ros-pkg. Code is to make pioneer3dx.
 Modified by Tracy Davies for this pkg-->
-<robot name="pioneer3dx"
-  xmlns:sensor="http://playerstage.sourceforge.net/gazebo/xmlschema/#sensor"
-  xmlns:controller="http://playerstage.sourceforge.net/gazebo/xmlschema/#controller"
-  xmlns:interface="http://playerstage.sourceforge.net/gazebo/xmlschema/#interface"
-  xmlns:xacro="http://ros.org/wiki/xacro">
+<robot name="pioneer3dx" xmlns:xacro="http://ros.org/wiki/xacro">
   <xacro:include filename="$(find p3dx_description)/defs/pioneer3dx_wheel.xacro"/>
 <!-- Chassis -->
@@ -166,4 +162,11 @@
 	</collision>
 	</link>
+  <gazebo reference="center_wheel">
+    <material value="Gazebo/Black"/>
+    <elem key="mu1" value="10.0" />
+    <elem key="mu2" value="10.0" />
+    <elem key="kp"  value="1000000.0" />
+    <elem key="kd"  value="1.0" />
+  </gazebo>
 	<joint name="center_wheel_joint" type="fixed">
 		<origin xyz="-0.0035 0 -0.001" rpy="0 0 0"/>
@@ -171,11 +174,4 @@
 		<child link="center_hubcap"/>
 	</joint>
-	<gazebo reference="center_wheel">
-		<material value="Gazebo/Black"/>
-    <elem key="mu1" value="10.0" />
-    <elem key="mu2" value="10.0" />
-    <elem key="kp"  value="1000000.0" />
-    <elem key="kd"  value="1.0" />
-	</gazebo>
 <xacro:p3dx_wheel suffix="left" parent="base_link" reflect="1"/>
 <xacro:p3dx_wheel suffix="right" parent="base_link" reflect="-1"/>
@@ -212,5 +208,5 @@
 		<child link="front_sonar"/>
 	</joint>
-	<link name="back_sonar">
+<!-- 	<link name="back_sonar">
 		<inertial>
 			<mass value="0.0001"/>
@@ -242,6 +238,6 @@
 		<parent link="base_link"/>
 		<child link="back_sonar"/>
-	</joint>
-  <gazebo>
+	</joint> -->
+<!--   <gazebo>
     <controller:differential_position2d name="controller1">
       <update>100</update>
@@ -260,11 +256,11 @@
       <gaussianNoise>0.01</gaussianNoise>
       <frameName>map</frameName>
-      <xyzOffsets>0 0 0</xyzOffsets> <!-- initialize odometry for fake localization-->
+      <xyzOffsets>0 0 0</xyzOffsets> initialize odometry for fake localization
       <rpyOffsets>0 0 0</rpyOffsets>
       <interface:position name="p3d_base_position"/>
     </controller:gazebo_ros_p3d>
-    <!-- this publishes empty joint_states due to no transmission, but
+    this publishes empty joint_states due to no transmission, but
          triggering robot_state_puublisher to publish tf between fixed joints in erratic,
-         (e.g. base_laser_link for the base_scan frame) -->
+         (e.g. base_laser_link for the base_scan frame)
     <controller:gazebo_ros_controller_manager name="gazebo_ros_controller_manager" plugin="libgazebo_ros_controller_manager.so">
       <alwaysOn>true</alwaysOn>
@@ -272,4 +268,4 @@
       <interface:audio name="gazebo_ros_controller_manager_dummy_iface" />
     </controller:gazebo_ros_controller_manager>
-  </gazebo>
+  </gazebo> -->
 </robot>

File: urdf/pioneer3dx.xacro.urdf (robot description, URDF)
Before this commit: robot pioneer3dx, 11 links, 10 joints
Links:
- removed link back_sonar
Joints:
- removed joint base_back_joint
