Commit message: Working model in rviz and gazebo; sonars are at wrong side.

File: urdf/pioneer3dx.xacro (robot description, xacro)
@@ -1,172 +1,165 @@
 <?xml version="1.0"?>
-<!-- Orignal in ucs-ros-pkg. Code is to make pioneer3dx.
-Modified by Tracy Davies for this pkg-->
+<!--
+This is the xacro description of a Pioneer 3DX, to be used in rviz and gazebo.
+Copyright (C) 2013 Rafael Berkvens rafael.berkvens@uantwerpen.be
+This program is free software: you can redistribute it and/or modify
+it under the terms of the GNU General Public License as published by
+the Free Software Foundation, either version 3 of the License, or
+(at your option) any later version.
+This program is distributed in the hope that it will be useful,
+but WITHOUT ANY WARRANTY; without even the implied warranty of
+MERCHANTABILITY or FITNESS FOR A PARTICULAR PURPOSE.  See the
+GNU General Public License for more details.
+You should have received a copy of the GNU General Public License
+along with this program.  If not, see <http://www.gnu.org/licenses/>.
+This project is based on work by Tracy Davies, where it was in turn based on
+work original in ucs-ros-pkg.
+ -->
 <robot name="pioneer3dx" xmlns:xacro="http://ros.org/wiki/xacro">
-  <xacro:include filename="$(find p3dx_description)/defs/pioneer3dx_wheel.xacro"/>
-<!-- Chassis -->
+  <!-- import all gazebo-customization elements, including gazebo colors -->
+  <xacro:include filename="$(find p3dx_description)/urdf/pioneer3dx.gazebo" />
+  <!-- import the pioneer 3dx's wheels -->
+  <xacro:include filename="$(find p3dx_description)/urdf/pioneer3dx_wheel.xacro" />
+  <!-- chassis -->
 	<link name="base_link">
 		<inertial>
-			<mass value="3.5"/>
-			<!--<origin xyz="-0.025 0 -0.223"/>-->
-			<origin xyz="-0.05 0 0"/>
-			<inertia ixx="1" ixy="0" ixz="0"
-				 iyy="1" iyz="0"
-				 izz="1"/>
+			<mass value="3.5" />
+			<!--<origin xyz="-0.025 0 -0.223"/> -->
+			<origin xyz="-0.05 0 0" />
+			<inertia ixx="1" ixy="0" ixz="0" iyy="1" iyz="0" izz="1" />
 		</inertial>
 		<visual name="base_visual">
-			<origin xyz="-0.045 0 0.148" rpy="0 0 0"/>
+			<origin xyz="-0.045 0 0.148" rpy="0 0 0" />
 			<geometry name="pioneer_geom">
-				<mesh filename="package://p3dx_description/meshes/chassis.stl"/>
+				<mesh filename="package://p3dx_description/meshes/chassis.stl" />
 			</geometry>
 			<material name="ChassisRed">
-				<color rgba="0.851 0.0 0.0 1.0"/>
+				<color rgba="0.851 0.0 0.0 1.0" />
 			</material>
 		</visual>
 		<collision>
-			<origin xyz="-0.045 0 0.145" rpy="0 0 0"/>
-				<geometry>
-					<box size="0.35 0.25 0.14"/>
-				</geometry>
+			<origin xyz="-0.045 0 0.145" rpy="0 0 0" />
+			<geometry>
+				<box size="0.35 0.25 0.14" />
+			</geometry>
 		</collision>
 	</link>
-	<gazebo reference="base_link">
-		<material value="Gazebo/Red"/>
-	</gazebo>
-<!-- Top -->
+  <!-- top_plate -->
 	<link name="top_plate">
 		<inertial>
-			<mass value="0.01"/>
-			<origin xyz="0 0 0"/>
-			<inertia ixx="1" ixy="0" ixz="0"
-				 iyy="1" iyz="0"
- 				izz="1"/>
+			<mass value="0.01" />
+			<origin xyz="0 0 0" />
+			<inertia ixx="1" ixy="0" ixz="0" iyy="1" iyz="0" izz="1" />
 		</inertial>
 		<visual name="base_visual">
-			<origin xyz="0 0 0" rpy="0 0 0"/>
+			<origin xyz="0 0 0" rpy="0 0 0" />
 			<geometry name="top_geom">
-				<mesh filename="package://p3dx_description/meshes/top.stl"/>
+				<mesh filename="package://p3dx_description/meshes/top.stl" />
 			</geometry>
 			<material name="TopBlack">
-					<color rgba="0.038 0.038 0.038 1.0"/>
+				<color rgba="0.038 0.038 0.038 1.0" />
 			</material>
 		</visual>
 		<collision>
-			<origin xyz="0.0 0 0" rpy="0 0 0"/>
+			<origin xyz="0.0 0 0" rpy="0 0 0" />
 			<geometry name="pioneer_geom">
-				<box size="0.45 0.38 0.01"/>
+				<box size="0.45 0.38 0.01" />
 			</geometry>
 		</collision>
 	</link>
-	<gazebo reference="top_plate">
-		<material value="Gazebo/Black"/>
-	</gazebo>
 	<joint name="base_top_joint" type="fixed">
-		<origin xyz="-0.045 0 0.234" rpy="0 0 0"/>
-		<parent link="base_link"/>
-		<child link="top_plate"/>
+		<origin xyz="-0.045 0 0.234" rpy="0 0 0" />
+		<parent link="base_link" />
+		<child link="top_plate" />
 	</joint>
-<!-- Swivel -->
+  <!-- swivel -->
 	<link name="swivel">
 		<inertial>
-			<mass value="0.1"/>
-			<origin xyz="0 0 0"/>
-			<inertia ixx="0.01" ixy="0" ixz="0"
-				 iyy="0.01" iyz="0" izz="0.01"/>
-  	 	</inertial>
-	<visual name="base_visual">
-		<origin xyz="0 0 0" rpy="0 0 0"/>
-		<geometry name="pioneer_geom">
-			<mesh filename="package://p3dx_description/meshes/swivel.stl"/>
-		</geometry>
-		<material name="swivel">
-			<color rgba="0.5 0.5 0.5 1"/>
-		</material>
-	</visual>
-	<collision>
-		<origin xyz="0 0 0" rpy="0 0 0"/>
-		<geometry>
-			<box size="0 0 0"/>
-		</geometry>
-	</collision>
+			<mass value="0.1" />
+			<origin xyz="0 0 0" />
+			<inertia ixx="0.01" ixy="0" ixz="0" iyy="0.01" iyz="0" izz="0.01" />
+		</inertial>
+		<visual name="base_visual">
+			<origin xyz="0 0 0" rpy="0 0 0" />
+			<geometry name="pioneer_geom">
+				<mesh filename="package://p3dx_description/meshes/swivel.stl" />
+			</geometry>
+			<material name="swivel">
+				<color rgba="0.5 0.5 0.5 1" />
+			</material>
+		</visual>
+		<collision>
+			<origin xyz="0 0 0" rpy="0 0 0" />
+			<geometry>
+				<box size="0 0 0" />
+			</geometry>
+		</collision>
 	</link>
-	<gazebo reference="swivel">
-		<material value="Gazebo/Grey"/>
-	</gazebo>
- 	<joint name="base_swivel_joint" type="continuous">
-		<origin xyz="-0.185 0 0.055" rpy="0 0 0"/>
-		<axis xyz="0 0 1"/>
-		<anchor xyz="0 0 0"/>
-    <limit effort="100" velocity="100" k_velocity="0" />
-    <joint_properties damping="0.0" friction="0.0" />
-		<parent link="base_link"/>
-		<child link="swivel"/>
+	<joint name="base_swivel_joint" type="continuous">
+		<origin xyz="-0.185 0 0.055" rpy="0 0 0" />
+		<axis xyz="0 0 1" />
+		<anchor xyz="0 0 0" />
+		<limit effort="100" velocity="100" k_velocity="0" />
+		<joint_properties damping="0.0" friction="0.0" />
+		<parent link="base_link" />
+		<child link="swivel" />
 	</joint>
-<!-- Center Wheel + Hubcap -->
+  <!-- center_hubcap -->
 	<link name="center_hubcap">
 		<inertial>
-			<mass value="0.01"/>
-			<origin xyz="0 0 0"/>
+			<mass value="0.01" />
+			<origin xyz="0 0 0" />
 			<inertia ixx="0.012411765597" ixy="-0.000711733678" ixz="0.00050272983"
-				 iyy="0.015218160428" iyz="-0.000004273467" izz="0.011763977943"/>
-  	 	</inertial>
-	<visual name="base_visual">
-		<origin xyz="0 0 0" rpy="0 0 0"/>
-		<geometry name="pioneer_geom">
-			<mesh filename="package://p3dx_description/meshes/center_hubcap.stl"/>
-		</geometry>
-		<material name="swivel">
-			<color rgba="0.5 0.5 0.5 1"/>
-		</material>
-	</visual>
-	<collision>
-		<origin xyz="0 0 0" rpy="0 0 0"/>
-		<geometry>
-			<box size="0 0 0"/>
-		</geometry>
-	</collision>
+				iyy="0.015218160428" iyz="-0.000004273467" izz="0.011763977943" />
+		</inertial>
+		<visual name="base_visual">
+			<origin xyz="0 0 0" rpy="0 0 0" />
+			<geometry name="pioneer_geom">
+				<mesh filename="package://p3dx_description/meshes/center_hubcap.stl" />
+			</geometry>
+			<material name="swivel">
+				<color rgba="0.5 0.5 0.5 1" />
+			</material>
+		</visual>
+		<collision>
+			<origin xyz="0 0 0" rpy="0 0 0" />
+			<geometry>
+				<box size="0 0 0" />
+			</geometry>
+		</collision>
 	</link>
-	<gazebo reference="center_hubcap">
-		<material value="Gazebo/Grey"/>
-	</gazebo>
 	<joint name="swivel_hubcap_joint" type="continuous">
-		<origin xyz="-0.026 0 -0.016" rpy="0 0 0"/>
-		<axis xyz="0 1 0"/>
-		<anchor xyz="0 0 0"/>
-    <limit effort="100" velocity="100" k_velocity="0" />
-    <joint_properties damping="0.0" friction="0.0" />
-	  <parent link="swivel"/>
-		<child link="center_wheel"/>
+		<origin xyz="-0.026 0 -0.016" rpy="0 0 0" />
+		<axis xyz="0 1 0" />
+		<anchor xyz="0 0 0" />
+		<limit effort="100" velocity="100" k_velocity="0" />
+		<joint_properties damping="0.0" friction="0.0" />
+		<parent link="swivel" />
+		<child link="center_wheel" />
 	</joint>
+  <!-- center_wheel -->
 	<link name="center_wheel">
 		<inertial>
-			<mass value="0.1"/>
-			<origin xyz="0 0 0"/>
+			<mass value="0.1" />
+			<origin xyz="0 0 0" />
 			<inertia ixx="0.012411765597" ixy="-0.000711733678" ixz="0.00050272983"
-				 iyy="0.015218160428" iyz="-0.000004273467" izz="0.011763977943"/>
-  	 	</inertial>
-	<visual name="base_visual">
-		<origin xyz="0 0 0" rpy="0 0 0"/>
-		<geometry name="pioneer_geom">
-			<mesh filename="package://p3dx_description/meshes/center_wheel.stl"/>
-		</geometry>
-		<material name="WheelBlack">
-			<color rgba="0.117 0.117 0.117 1"/>
-		</material>
-	</visual>
-	<collision>
-		<origin xyz="0 0 0" rpy="${-3.1415927/2.0} 0 0"/>
-		<geometry>
-			<!--<mesh filename="package://p3dx_description/meshes/center_wheel.stl"/>-->
-			<cylinder radius="0.0375" length="0.01"/>
-		</geometry>
-	</collision>
+				iyy="0.015218160428" iyz="-0.000004273467" izz="0.011763977943" />
+		</inertial>
+		<visual name="base_visual">
+			<origin xyz="0 0 0" rpy="0 0 0" />
+			<geometry name="pioneer_geom">
+				<mesh filename="package://p3dx_description/meshes/center_wheel.stl" />
+			</geometry>
+			<material name="WheelBlack">
+				<color rgba="0.117 0.117 0.117 1" />
+			</material>
+		</visual>
+		<collision>
+			<origin xyz="0 0 0" rpy="${-3.1415927/2.0} 0 0" />
+			<geometry>
+				<cylinder radius="0.0375" length="0.01" />
+			</geometry>
+		</collision>
 	</link>
-  <gazebo reference="center_wheel">
-    <material value="Gazebo/Black"/>
-    <elem key="mu1" value="10.0" />
-    <elem key="mu2" value="10.0" />
-    <elem key="kp"  value="1000000.0" />
-    <elem key="kd"  value="1.0" />
-  </gazebo>
 	<joint name="center_wheel_joint" type="fixed">
 		<origin xyz="-0.0035 0 -0.001" rpy="0 0 0"/>
@@ -174,98 +167,33 @@
 		<child link="center_hubcap"/>
 	</joint>
-<xacro:p3dx_wheel suffix="left" parent="base_link" reflect="1"/>
-<xacro:p3dx_wheel suffix="right" parent="base_link" reflect="-1"/>
-<!-- Front + Back Sonar -->
+	<xacro:p3dx_wheel suffix="left" parent="base_link" reflect="1"/>
+	<xacro:p3dx_wheel suffix="right" parent="base_link" reflect="-1"/>
+  <!-- front_sonar -->
 	<link name="front_sonar">
 		<inertial>
-			<mass value="0.0001"/>
-			<origin xyz="0 0 0"/>
-			<inertia ixx="1" ixy="0" ixz="0"
-				 iyy="1" iyz="0" izz="1"/>
+			<mass value="0.0001" />
+			<origin xyz="0 0 0" />
+			<inertia ixx="1" ixy="0" ixz="0" iyy="1" iyz="0" izz="1" />
 		</inertial>
 		<visual name="base_visual">
-			<origin xyz="0 0 0" rpy="0 0 0"/>
+			<origin xyz="0 0 0" rpy="0 0 0" />
 			<geometry name="pioneer_geom">
-				<mesh filename="package://p3dx_description/meshes/front_sonar.stl"/>
+				<mesh filename="package://p3dx_description/meshes/front_sonar.stl" />
 			</geometry>
 			<material name="SonarYellow">
-				<color rgba="0.715 0.583 0.210 1.0"/>
+				<color rgba="0.715 0.583 0.210 1.0" />
 			</material>
 		</visual>
 		<collision>
-			<origin xyz="0 0 0" rpy="0 0 0"/>
+			<origin xyz="0 0 0" rpy="0 0 0" />
 			<geometry>
-				<box size="0 0 0"/>
+				<box size="0 0 0" />
 			</geometry>
 		</collision>
 	</link>
-	<gazebo reference="front_sonar">
-		<material value="Gazebo/Yellow"/>
-	</gazebo>
 	<joint name="base_front_joint" type="fixed">
-		<origin xyz="-0.198 0 0.208" rpy="0 0 0"/>
-		<parent link="base_link"/>
-		<child link="front_sonar"/>
+		<origin xyz="-0.198 0 0.208" rpy="0 0 0" />
+		<parent link="base_link" />
+		<child link="front_sonar" />
 	</joint>
-<!-- 	<link name="back_sonar">
-		<inertial>
-			<mass value="0.0001"/>
-			<origin xyz="0 0 0"/>
-			<inertia ixx="1" ixy="0" ixz="0"
-				 iyy="1" iyz="0" izz="1"/>
-		</inertial>
-		<visual name="back_sonar_vis">
-			<origin xyz="0 0 0" rpy="0 0 0"/>
-			<geometry name="pioneer_geom">
-				<mesh filename="package://p3dx_description/meshes/back_sonar.stl"/>
-			</geometry>
-			<material name="SonarYellow">
-				<color rgba="0.715 0.583 0.210 1.0"/>
-			</material>
-		</visual>
-		<collision>
-			<origin xyz="0 0 0" rpy="0 0 0"/>
-			<geometry>
-				<box size="0 0 0"/>
-			</geometry>
-		</collision>
-	</link>
-	<gazebo reference="back_sonar">
-		<material value="Gazebo/Yellow"/>
-	</gazebo>
-	<joint name="base_back_joint" type="fixed">
-		<origin xyz="0.109 0 0.209" rpy="0 0 0"/>
-		<parent link="base_link"/>
-		<child link="back_sonar"/>
-	</joint> -->
-<!--   <gazebo>
-    <controller:differential_position2d name="controller1">
-      <update>100</update>
-      <leftJoint>base_right_wheel_joint</leftJoint>
-      <rightJoint>base_left_wheel_joint</rightJoint>
-      <wheelSeparation>0.39</wheelSeparation>
-      <wheelDiameter>0.15</wheelDiameter>
-      <torque>5</torque>
-      <interface:position name="position_iface_0"/>
-    </controller:differential_position2d>
-    <controller:gazebo_ros_p3d name="p3d_base_controller" plugin="libgazebo_ros_p3d.so">
-      <alwaysOn>true</alwaysOn>
-      <updateRate>100.0</updateRate>
-      <bodyName>base_link</bodyName>
-      <topicName>base_pose_ground_truth</topicName>
-      <gaussianNoise>0.01</gaussianNoise>
-      <frameName>map</frameName>
-      <xyzOffsets>0 0 0</xyzOffsets> initialize odometry for fake localization
-      <rpyOffsets>0 0 0</rpyOffsets>
-      <interface:position name="p3d_base_position"/>
-    </controller:gazebo_ros_p3d>
-    this publishes empty joint_states due to no transmission, but
-         triggering robot_state_puublisher to publish tf between fixed joints in erratic,
-         (e.g. base_laser_link for the base_scan frame)
-    <controller:gazebo_ros_controller_manager name="gazebo_ros_controller_manager" plugin="libgazebo_ros_controller_manager.so">
-      <alwaysOn>true</alwaysOn>
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